File: KiCad/Beerator/Beerator.kicad_sch (KiCad schematic)
At the start: 0 parts

Commit message: feat(last pcb version)
Parts:
- added H101, H102, H103, H104: MountingHole_Pad, MountingHole:MountingHole_3.2mm_M3_Pad_Via, symbol Mechanical:MountingHole_Pad
Connections:
- new net GND: H101.1, H102.1, H103.1, H104.1
