File: KiCad/Beerator/actuator_bloc.kicad_sch (KiCad schematic)
At the start: 16 parts, among them U5 Servo

Commit message: feat(KiCad): Version 2
Connections:
- net 01_D1 is gone; now on net O1_D1: JMCC1_0.6 (Pin_6)
- net 02_D1 is gone; now on net O2_D1: JMCC1_0.5 (Pin_5)
- net GND: now also C201.1, C202.1, UDRIVER1.2 (VM), UDRIVER2.2 (VM)
- net 01_D2 renamed O1_D2
- net 02_D2 renamed O2_D2
Changed lines of the file:
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@@
   (junction (at 77.47 110.49) (diameter 0) (color 0 0 0 0)
   )
+  (junction (at 77.47 110.617) (diameter 0) (color 0 0 0 0)
+  )
   (junction (at 77.47 114.3) (diameter 0) (color 0 0 0 0)
   )
@@
   (junction (at 73.66 38.1) (diameter 0) (color 0 0 0 0)
   )
+  (junction (at 78.74 38.1) (diameter 0) (color 0 0 0 0)
+  )
+  (junction (at 82.55 110.617) (diameter 0) (color 0 0 0 0)
+  )
   (junction (at 160.02 130.81) (diameter 0) (color 0 0 0 0)
   )
@@
     (stroke (width 0) (type default) (color 0 0 0 0))
   )
-  (wire (pts (xy 77.47 110.49) (xy 77.47 114.3))
+  (wire (pts (xy 77.47 110.49) (xy 77.47 110.617))
     (stroke (width 0) (type default) (color 0 0 0 0))
   )
@@
     (stroke (width 0) (type default) (color 0 0 0 0))
   )
-  (wire (pts (xy 82.55 110.49) (xy 82.55 115.57))
+  (wire (pts (xy 82.55 110.49) (xy 82.55 110.617))
     (stroke (width 0) (type default) (color 0 0 0 0))
   )
@@
     (stroke (width 0) (type default) (color 0 0 0 0))
   )
+  (wire (pts (xy 77.47 110.617) (xy 77.47 114.3))
+    (stroke (width 0) (type default) (color 0 0 0 0))
+  )
   (wire (pts (xy 153.67 86.36) (xy 157.48 86.36))
     (stroke (width 0) (type default) (color 0 0 0 0))
@@
     (stroke (width 0) (type default) (color 0 0 0 0))
   )
+  (wire (pts (xy 82.55 110.617) (xy 82.55 115.57))
+    (stroke (width 0) (type default) (color 0 0 0 0))
+  )
   (wire (pts (xy 77.47 100.33) (xy 77.47 110.49))
     (stroke (width 0) (type default) (color 0 0 0 0))
@@
     (stroke (width 0) (type default) (color 0 0 0 0))
   )
+  (wire (pts (xy 77.47 110.617) (xy 82.55 110.617))
+    (stroke (width 0) (type default) (color 0 0 0 0))
+  )
   (wire (pts (xy 49.53 123.19) (xy 49.53 134.62))
     (stroke (width 0) (type default) (color 0 0 0 0))
@@
   )
   (wire (pts (xy 152.4 96.52) (xy 157.48 96.52))
+    (stroke (width 0) (type default) (color 0 0 0 0))
+  )
+  (wire (pts (xy 73.66 38.1) (xy 78.74 38.1))
     (stroke (width 0) (type default) (color 0 0 0 0))
   )
@@
     )
   )
-  (global_label "01_D1" (shape input) (at 149.86 35.56 180) (fields_autoplaced)
-    (effects (font (size 1.27 1.27)) (justify right))
-    (property "Intersheet References" "${INTERSHEET_REFS}" (id 0) (at 141.5807 35.4806 0)
+  (global_label "O1_D1" (shape input) (at 149.86 35.56 180) (fields_autoplaced)
+    (effects (font (size 1.27 1.27)) (justify right))
+    (property "Intersheet References" "${INTERSHEET_REFS}" (id 0) (at 141.4598 35.4806 0)
       (effects (font (size 1.27 1.27)) (justify right) hide)
     )
@@
     )
   )
-  (global_label "01_D2" (shape input) (at 153.67 83.82 180) (fields_autoplaced)
-    (effects (font (size 1.27 1.27)) (justify right))
-    (property "Intersheet References" "${INTERSHEET_REFS}" (id 0) (at 145.3907 83.7406 0)
+  (global_label "O1_D2" (shape input) (at 153.67 83.82 180) (fields_autoplaced)
+    (effects (font (size 1.27 1.27)) (justify right))
+    (property "Intersheet References" "${INTERSHEET_REFS}" (id 0) (at 145.2698 83.7406 0)
       (effects (font (size 1.27 1.27)) (justify right) hide)
     )
@@
     )
   )
-  (global_label "01_D2" (shape input) (at 90.17 123.19 0) (fields_autoplaced)
-    (effects (font (size 1.27 1.27)) (justify left))
-    (property "Intersheet References" "${INTERSHEET_REFS}" (id 0) (at 98.4493 123.1106 0)
+  (global_label "O1_D2" (shape input) (at 90.17 123.19 0) (fields_autoplaced)
+    (effects (font (size 1.27 1.27)) (justify left))
+    (property "Intersheet References" "${INTERSHEET_REFS}" (id 0) (at 98.5702 123.1106 0)
       (effects (font (size 1.27 1.27)) (justify left) hide)
     )
@@
     )
   )
-  (global_label "02_D2" (shape input) (at 90.17 128.27 0) (fields_autoplaced)
-    (effects (font (size 1.27 1.27)) (justify left))
-    (property "Intersheet References" "${INTERSHEET_REFS}" (id 0) (at 98.4493 128.1906 0)
-      (effects (font (size 1.27 1.27)) (justify left) hide)
-    )
-  )
-  (global_label "02_D2" (shape input) (at 153.67 86.36 180) (fields_autoplaced)
-    (effects (font (size 1.27 1.27)) (justify right))
-    (property "Intersheet References" "${INTERSHEET_REFS}" (id 0) (at 145.3907 86.2806 0)
+  (global_label "O2_D2" (shape input) (at 90.17 128.27 0) (fields_autoplaced)
+    (effects (font (size 1.27 1.27)) (justify left))
+    (property "Intersheet References" "${INTERSHEET_REFS}" (id 0) (at 98.5702 128.1906 0)
+      (effects (font (size 1.27 1.27)) (justify left) hide)
+    )
+  )
+  (global_label "O2_D2" (shape input) (at 153.67 86.36 180) (fields_autoplaced)
+    (effects (font (size 1.27 1.27)) (justify right))
+    (property "Intersheet References" "${INTERSHEET_REFS}" (id 0) (at 145.2698 86.2806 0)
       (effects (font (size 1.27 1.27)) (justify right) hide)
     )
@@
     )
   )
-  (global_label "02_D1" (shape input) (at 149.86 38.1 180) (fields_autoplaced)
-    (effects (font (size 1.27 1.27)) (justify right))
-    (property "Intersheet References" "${INTERSHEET_REFS}" (id 0) (at 141.5807 38.0206 0)
-      (effects (font (size 1.27 1.27)) (justify right) hide)
-    )
+  (global_label "O2_D1" (shape input) (at 149.86 38.1 180) (fields_autoplaced)
+    (effects (font (size 1.27 1.27)) (justify right))
+    (property "Intersheet References" "${INTERSHEET_REFS}" (id 0) (at 141.4598 38.0206 0)
+      (effects (font (size 1.27 1.27)) (justify right) hide)
+    )

Commit message: feat(last pcb version)
Parts:
- added C206: 100uF, Capacitor_THT:CP_Radial_D5.0mm_P2.00mm, symbol Device:C_Polarized_Small_US
- added C207, C208, C209, C210: 0.1uF, Capacitor_SMD:C_0603_1608Metric_Pad1.08x0.95mm_HandSolder, symbol Device:C_Small
- added JP3, JP4, JP5, JP6: SolderJumper_2_Open, Jumper:SolderJumper-3_P2.0mm_Open_TrianglePad1.0x1.5mm, symbol Jumper:SolderJumper_2_Open
- added R205: 10k, Resistor_SMD:R_0603_1608Metric_Pad0.98x0.95mm_HandSolder, symbol Device:R_Small
- C201, C202: footprint Capacitor_SMD:C_0603_1608Metric_Pad1.08x0.95mm_HandSolder -> Capacitor_THT:CP_Radial_D5.0mm_P2.00mm
- C204, C205: value 10µF -> 1µF
- JMCC1_0, JMCC2_0: footprint Connector_JST:JST_EH_B6B-EH-A_1x06_P2.50mm_Vertical -> Connector_JST:JST_XH_B6B-XH-AM_1x06_P2.50mm_Vertical
- JSERVO0: footprint Connector_JST:JST_XA_B03B-XASK-1-A_1x03_P2.50mm_Vertical -> Connector_JST:JST_XH_B3B-XH-AM_1x03_P2.50mm_Vertical
Connections:
- net 5: now also C204.2, C205.2, UDRIVER1.3 (VDD), UDRIVER2.3 (VDD), R205.2
- net GND: now also C206.2, C207.1, C208.1, C209.1, C210.1; no longer C201.1, C202.1, C203.2, C204.2, C205.2, JSERVO0.3 (Pin_3), UDRIVER1.2 (VM), UDRIVER1.3 (VDD), UDRIVER2.2 (VM), UDRIVER2.3 (VDD)
- net O1_D1: now also C210.2, JP3.2 (B); no longer UDRIVER1.1 (OUT1)
- net O1_D2: now also JMCC2_0.5 (Pin_5), C208.2, JP5.2 (B); no longer JMCC2_0.6 (Pin_6), UDRIVER2.1 (OUT1)
- net O2_D1: now also C209.2, JP4.2 (B); no longer UDRIVER1.7 (OUT2)
- net O2_D2: now also JMCC2_0.6 (Pin_6), C207.2, JP6.2 (B); no longer JMCC2_0.5 (Pin_5), UDRIVER2.7 (OUT2)
- net PHASE_A_M2: now also JMCC2_0.1 (Pin_1); no longer JMCC2_0.2 (Pin_2)
- net PHASE_B_M2: now also JMCC2_0.2 (Pin_2); no longer JMCC2_0.1 (Pin_1)
- net SERVO_DATA: now also R205.1
- new net: JP6.1 (A), UDRIVER2.7 (OUT2)
- new net: JP3.1 (A), UDRIVER1.1 (OUT1)
- new net: JP4.1 (A), UDRIVER1.7 (OUT2)
- new net: JP5.1 (A), UDRIVER2.1 (OUT1)
- new net 7.2: C201.1, C202.1, C203.2, C206.1, JSERVO0.3 (Pin_3), UDRIVER1.2 (VM), UDRIVER2.2 (VM)
Other:
- note added: "C201 : Chimique pour la puissance C205 : Ceramique"
- note added: "C202 : Chimique C204 : Ceramique"
- note added: "C206 : Chimique C203 : Ceramique"

Commit message: Update_Schemas
Parts:
- removed C209, C210: 0.1uF, Capacitor_SMD:C_0603_1608Metric_Pad1.08x0.95mm_HandSolder, symbol Device:C_Small
- removed JMCC1_0: Conn_01x06_Female, Connector_JST:JST_XH_B6B-XH-AM_1x06_P2.50mm_Vertical, symbol Connector:Conn_01x06_Female
- removed JMCC1_1: Conn_01x06_Female, symbol Connector:Conn_01x06_Female
- removed UMCC1: FIT0521, symbol Projet_Lib:FIT0521
- added C508, C510: 0.1uF, Capacitor_SMD:C_0603_1608Metric_Pad1.08x0.95mm_HandSolder, symbol Device:C_Small
- added JMCC0_502: Conn_01x06_Female, Connector_JST:JST_XH_B6B-XH-AM_1x06_P2.50mm_Vertical, symbol Connector:Conn_01x06_Female
- added JMCC0_504: Conn_01x06_Female, symbol Connector:Conn_01x06_Female
- added UMCC0_502: FIT0521, symbol Projet_Lib:FIT0521
- renumbered C205 to C501, C204 to C502, C201 to C503, C202 to C504, C206 to C505, C207 to C506, C203 to C507, C208 to C509, JMCC2_0 to JMCC1_501, JMCC2_1 to JMCC1_503, JP3 to JP501, JP4 to JP502, JP5 to JP503, JP6 to JP504, JSERVO0 to JSERVO501, JSERVO1 to JSERVO502, R205 to R501, U5 to U501, UDRIVER1 to UDRIVER501, UDRIVER2 to UDRIVER502, UMCC2 to UMCC1_501
Connections:
- net GND: now also JMCC1_501.5 (Pin_5), JSERVO501.3 (Pin_3), C508.1, C510.1, JMCC0_502.5 (Pin_5); no longer JMCC1_501.3 (Pin_3), JSERVO501.1 (Pin_1)
- net O1_D1: now also C510.2, JMCC0_502.1 (Pin_1)
- net O1_D2: now also JMCC1_501.1 (Pin_1); no longer JMCC1_501.5 (Pin_5)
- net O2_D1: now also C508.2, JMCC0_502.6 (Pin_6)
- net PHASE_A_M1: now also JMCC0_502.4 (Pin_4)
- net PHASE_A_M2: now also JMCC1_501.4 (Pin_4); no longer JMCC1_501.1 (Pin_1)
- net PHASE_B_M1: now also JMCC0_502.3 (Pin_3)
- net PHASE_B_M2: now also JMCC1_501.3 (Pin_3); no longer JMCC1_501.2 (Pin_2)
- net SERVO_DATA: now also JSERVO501.1 (Pin_1); no longer JSERVO501.2 (Pin_2)
- net 5 renamed +5V
- net +5V: now also JMCC1_501.2 (Pin_2), JMCC0_502.2 (Pin_2); no longer JMCC1_501.4 (Pin_4)
- net 7.2 renamed +BATT
- net +BATT: now also JSERVO501.2 (Pin_2); no longer JSERVO501.3 (Pin_3)
- new net: JMCC0_504.1 (Pin_1), UMCC0_502. (M-)
- new net: JMCC0_504.2 (Pin_2), UMCC0_502. (M-)
- new net: JMCC0_504.3 (Pin_3), UMCC0_502. (M-)
- new net: JMCC0_504.4 (Pin_4), UMCC0_502. (M-)
- new net: JMCC0_504.5 (Pin_5), UMCC0_502. (M-)
- new net: JMCC0_504.6 (Pin_6), UMCC0_502. (M-)
Other:
- moved on the sheet: C505, C506, C507, C509, R501, UMCC1_501

Commit message: pcb_v2
Changed lines of the file:
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@@
   (symbol (lib_id "Jumper:SolderJumper_2_Open") (at 96.52 128.27 0) (unit 1)
     (in_bom yes) (on_board yes)
-    (property "Reference" "JP504" (id 0) (at 96.52 125.73 0))
+    (property "Reference" "JP504" (id 0) (at 96.52 126.238 0))
     (property "Value" "SolderJumper_2_Open" (id 1) (at 97.79 130.81 0))
     (property "Footprint" "Jumper:SolderJumper-3_P2.0mm_Open_TrianglePad1.0x1.5mm" (id 2) (at 96.52 128.27 0)

Commit message: version_finale_pcb
Parts:
- JP501, JP502, JP503, JP504: footprint Jumper:SolderJumper-3_P2.0mm_Open_TrianglePad1.0x1.5mm -> Jumper:SolderJumper-2_P1.3mm_Open_Pad1.0x1.5mm
- renumbered JMCC0_502 to JMCC0_501, JMCC0_504 to JMCC0_502, JMCC1_503 to JMCC1_502, UMCC0_502 to UMCC0_501
Connections:
- net +5V: no longer R501.2
- new net +3.3V: R501.2
Changed lines of the file:
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@@
     (stroke (width 0) (type default) (color 0 0 0 0))
   )
-  (wire (pts (xy 153.67 139.7) (xy 152.4 139.7))
+  (wire (pts (xy 151.8412 139.7) (xy 153.67 139.7))
     (stroke (width 0) (type default) (color 0 0 0 0))
   )
@@
     (property "Reference" "JP504" (id 0) (at 96.52 126.238 0))
     (property "Value" "SolderJumper_2_Open" (id 1) (at 97.79 130.81 0))
-    (property "Footprint" "Jumper:SolderJumper-3_P2.0mm_Open_TrianglePad1.0x1.5mm" (id 2) (at 96.52 128.27 0)
+    (property "Footprint" "Jumper:SolderJumper-2_P1.3mm_Open_Pad1.0x1.5mm" (id 2) (at 96.52 128.27 0)
       (effects (font (size 1.27 1.27)) hide)
     )
@@
   (symbol (lib_name "FIT0521_1") (lib_id "Projet_Lib:FIT0521") (at 212.09 44.45 0) (unit 1)
     (in_bom yes) (on_board yes) (fields_autoplaced)
-    (property "Reference" "UMCC0_502" (id 0) (at 222.25 36.8299 0)
+    (property "Reference" "UMCC0_501" (id 0) (at 222.25 36.8299 0)
       (effects (font (size 1.27 1.27)) (justify left))
     )
@@
   (symbol (lib_id "Connector:Conn_01x06_Female") (at 168.91 39.37 0) (mirror x) (unit 1)
     (in_bom yes) (on_board yes)
-    (property "Reference" "JMCC0_502" (id 0) (at 163.83 29.21 0))
+    (property "Reference" "JMCC0_501" (id 0) (at 163.83 29.21 0))
     (property "Value" "Conn_01x06_Female" (id 1) (at 163.83 26.67 0))
     (property "Footprint" "Connector_JST:JST_XH_B6B-XH-AM_1x06_P2.50mm_Vertical" (id 2) (at 168.91 39.37 0)
@@
     (property "Reference" "JP503" (id 0) (at 96.52 120.65 0))
     (property "Value" "SolderJumper_2_Open" (id 1) (at 97.79 125.73 0))
-    (property "Footprint" "Jumper:SolderJumper-3_P2.0mm_Open_TrianglePad1.0x1.5mm" (id 2) (at 96.52 123.19 0)
+    (property "Footprint" "Jumper:SolderJumper-2_P1.3mm_Open_Pad1.0x1.5mm" (id 2) (at 96.52 123.19 0)
       (effects (font (size 1.27 1.27)) hide)
     )
@@
     (property "Reference" "JP502" (id 0) (at 92.71 59.69 0))
     (property "Value" "SolderJumper_2_Open" (id 1) (at 93.98 57.15 0))
-    (property "Footprint" "Jumper:SolderJumper-3_P2.0mm_Open_TrianglePad1.0x1.5mm" (id 2) (at 92.71 54.61 0)
+    (property "Footprint" "Jumper:SolderJumper-2_P1.3mm_Open_Pad1.0x1.5mm" (id 2) (at 92.71 54.61 0)
       (effects (font (size 1.27 1.27)) hide)
     )
@@
   (symbol (lib_id "Connector:Conn_01x06_Female") (at 180.34 39.37 180) (unit 1)
     (in_bom yes) (on_board yes)
-    (property "Reference" "JMCC0_504" (id 0) (at 186.69 22.86 0))
+    (property "Reference" "JMCC0_502" (id 0) (at 186.69 22.86 0))
     (property "Value" "Conn_01x06_Female" (id 1) (at 184.15 25.4 0))
     (property "Footprint" "" (id 2) (at 180.34 39.37 0)
@@
   (symbol (lib_id "power:+5V") (at 152.4 93.98 90) (unit 1)
     (in_bom yes) (on_board yes) (fields_autoplaced)
-    (property "Reference" "#PWR0520" (id 0) (at 156.21 93.98 0)
+    (property "Reference" "#PWR0521" (id 0) (at 156.21 93.98 0)
       (effects (font (size 1.27 1.27)) hide)
     )
@@
     )
     (property "Datasheet" "" (id 3) (at 134.62 91.44 0)
+      (effects (font (size 1.27 1.27)) hide)
+    )
+    (pin "1")
+  )
+  (symbol (lib_id "power:+3.3V") (at 151.8412 139.7 90) (unit 1)
+    (in_bom yes) (on_board yes) (fields_autoplaced)
+    (property "Reference" "#PWR0520" (id 0) (at 155.6512 139.7 0)
+      (effects (font (size 1.27 1.27)) hide)
+    )
+    (property "Value" "+3.3V" (id 1) (at 148.0058 139.6999 90)
+      (effects (font (size 1.27 1.27)) (justify left))
+    )
+    (property "Footprint" "" (id 2) (at 151.8412 139.7 0)
+      (effects (font (size 1.27 1.27)) hide)
+    )
+    (property "Datasheet" "" (id 3) (at 151.8412 139.7 0)
       (effects (font (size 1.27 1.27)) hide)
     )
@@
     (property "Reference" "JP501" (id 0) (at 92.71 46.99 0))
     (property "Value" "SolderJumper_2_Open" (id 1) (at 93.98 52.07 0))
-    (property "Footprint" "Jumper:SolderJumper-3_P2.0mm_Open_TrianglePad1.0x1.5mm" (id 2) (at 92.71 49.53 0)
+    (property "Footprint" "Jumper:SolderJumper-2_P1.3mm_Open_Pad1.0x1.5mm" (id 2) (at 92.71 49.53 0)
       (effects (font (size 1.27 1.27)) hide)
     )
@@
   (symbol (lib_id "Connector:Conn_01x06_Female") (at 173.99 91.44 180) (unit 1)
     (in_bom yes) (on_board yes)
-    (property "Reference" "JMCC1_503" (id 0) (at 180.34 74.93 0))
+    (property "Reference" "JMCC1_502" (id 0) (at 180.34 74.93 0))
     (property "Value" "Conn_01x06_Female" (id 1) (at 177.8 77.47 0))
     (property "Footprint" "" (id 2) (at 173.99 91.44 0)
@@
       (effects (font (size 1.27 1.27)) hide)
     )
-    (pin "1")
-  )
-  (symbol (lib_id "power:+5V") (at 152.4 139.7 90) (unit 1)
-    (in_bom yes) (on_board yes)
-    (property "Reference" "#PWR0521" (id 0) (at 156.21 139.7 0)
-      (effects (font (size 1.27 1.27)) hide)
-    )
-    (property "Value" "+5V" (id 1) (at 148.59 140.97 0))
-    (property "Footprint" "" (id 2) (at 152.4 139.7 0)
-      (effects (font (size 1.27 1.27)) hide)
-    )
-    (property "Datasheet" "" (id 3) (at 152.4 139.7 0)
-      (effects (font (size 1.27 1.27)) hide)
-    )
