File: KiCad/Beerator/sensor_bloc.kicad_sch (KiCad schematic)
At the start: 12 parts

Commit message: feat(KiCad): Version 2
Connections:
- no-connect marks 0 -> 1
Changed lines of the file:
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@@
   (junction (at 50.8 40.64) (diameter 0) (color 0 0 0 0)
   )
+  (no_connect (at 243.205 36.83))
   (wire (pts (xy 187.96 48.26) (xy 199.39 48.26))
     (stroke (width 0) (type default) (color 0 0 0 0))
@@
     (stroke (width 0) (type default) (color 0 0 0 0))
   )
+  (wire (pts (xy 243.205 36.83) (xy 247.65 36.83))
+    (stroke (width 0) (type default) (color 0 0 0 0))
+  )
   (polyline (pts (xy 11.43 86.36) (xy 171.45 86.36))
     (stroke (width 0) (type default) (color 0 0 0 0))
@@
     (stroke (width 0) (type default) (color 0 0 0 0))
   )
+  (wire (pts (xy 43.561 172.72) (xy 55.88 172.72))
+    (stroke (width 0) (type default) (color 0 0 0 0))
+  )
   (wire (pts (xy 74.93 50.8) (xy 81.28 50.8))
     (stroke (width 0) (type default) (color 0 0 0 0))
@@
     (stroke (width 0) (type default) (color 0 0 0 0))
   )
-  (polyline (pts (xy 10.16 140.97) (xy 170.18 142.24))
+  (polyline (pts (xy 10.16 140.97) (xy 170.434 140.589))
     (stroke (width 0) (type default) (color 0 0 0 0))
   )
@@
     (stroke (width 0) (type default) (color 0 0 0 0))
   )
-  (polyline (pts (xy 171.45 78.74) (xy 171.45 86.36))
-    (stroke (width 0) (type default) (color 0 0 0 0))
-  )
   (wire (pts (xy 85.09 135.89) (xy 144.78 135.89))
     (stroke (width 0) (type default) (color 0 0 0 0))
@@
     (stroke (width 0) (type default) (color 0 0 0 0))
   )
+  (wire (pts (xy 45.466 118.11) (xy 52.07 118.11))
+    (stroke (width 0) (type default) (color 0 0 0 0))
+  )
   (wire (pts (xy 44.45 45.72) (xy 50.8 45.72))
     (stroke (width 0) (type default) (color 0 0 0 0))
@@
     (stroke (width 0) (type default) (color 0 0 0 0))
   )
-  (polyline (pts (xy 171.45 86.36) (xy 170.18 142.24))
+  (polyline (pts (xy 170.434 86.233) (xy 170.434 140.589))
     (stroke (width 0) (type default) (color 0 0 0 0))
   )
@@
     )
   )
-  (global_label "IR1-OUT" (shape input) (at 52.07 118.11 180) (fields_autoplaced)
-    (effects (font (size 1.27 1.27)) (justify right))
-    (property "Intersheet References" "${INTERSHEET_REFS}" (id 0) (at 41.3717 118.0306 0)
-      (effects (font (size 1.27 1.27)) (justify right) hide)
-    )
-  )
-  (global_label "IR2-OUT" (shape input) (at 55.88 172.72 180) (fields_autoplaced)
-    (effects (font (size 1.27 1.27)) (justify right))
-    (property "Intersheet References" "${INTERSHEET_REFS}" (id 0) (at 45.1817 172.6406 0)
-      (effects (font (size 1.27 1.27)) (justify right) hide)
-    )
+  (global_label "IR1-OUT" (shape input) (at 45.466 118.11 180) (fields_autoplaced)
+    (effects (font (size 1.27 1.27)) (justify right))
+    (property "Intersheet References" "${INTERSHEET_REFS}" (id 0) (at 34.7677 118.0306 0)
+      (effects (font (size 1.27 1.27)) (justify right) hide)
+    )
+  )
+  (global_label "IR2-OUT" (shape input) (at 43.561 172.72 180) (fields_autoplaced)
+    (effects (font (size 1.27 1.27)) (justify right))
+    (property "Intersheet References" "${INTERSHEET_REFS}" (id 0) (at 32.8627 172.6406 0)
+      (effects (font (size 1.27 1.27)) (justify right) hide)
+    )

Commit message: feat(last pcb version)
Parts:
- added JTOF1_0: Conn_01x06_Female, Connector_JST:JST_XH_B6B-XH-AM_1x06_P2.50mm_Vertical, symbol Connector:Conn_01x06_Female
- added JTOF1_1: Conn_01x06_Female, symbol Connector:Conn_01x06_Female
- added R301, R302, R303, R304: 1k, Resistor_SMD:R_0603_1608Metric_Pad0.98x0.95mm_HandSolder, symbol Device:R_Small
- added UTOF1: TOF-SENSOR-VL53LX, symbol Sensors_Beerator:TOF-SENSOR-VL53LX
- JCOLOR0: footprint Connector_JST:JST_EH_B7B-EH-A_1x07_P2.50mm_Vertical -> Connector_JST:JST_XH_B7B-XH-AM_1x07_P2.50mm_Vertical
- JDistance0_1: footprint Connector_JST:JST_EH_B3B-EH-A_1x03_P2.50mm_Vertical -> Connector_JST:JST_XH_B3B-XH-AM_1x03_P2.50mm_Vertical
- JDistance0_2: footprint (none) -> Connector_JST:JST_XH_B3B-XH-AM_1x03_P2.50mm_Vertical
- JDistance1_1: footprint Connector_JST:JST_EH_B3B-EH-A_1x03_P2.50mm_Vertical -> (none)
- JTOF0_0: renamed from JTOF0; footprint Connector_JST:JST_EH_B6B-EH-A_1x06_P2.50mm_Vertical -> Connector_JST:JST_XH_B6B-XH-AM_1x06_P2.50mm_Vertical
- renumbered JTOF1 to JTOF0_1
Connections:
- net 3.3: now also JTOF1_0.6 (Pin_6), R301.2, R302.2, R303.2, R304.2
- net GND: now also JTOF1_0.5 (Pin_5)
- net TOF-EXTI: now also JTOF0_0.4 (Pin_4); no longer JTOF0_0.2 (Pin_2)
- net TOF-SCL: now also JTOF0_0.2 (Pin_2), R304.1; no longer JTOF0_0.3 (Pin_3)
- net TOF-SDA: now also R303.1
- net TOF-XSHUT: now also JTOF0_0.3 (Pin_3); no longer JTOF0_0.4 (Pin_4)
- new net: JTOF1_1.1 (Pin_1), UTOF1.9 (SDA)
- new net: JTOF1_1.2 (Pin_2), UTOF1.7 (GPIO1)
- new net: JTOF1_1.3 (Pin_3), UTOF1.10 (SCL)
- new net: JTOF1_1.4 (Pin_4), UTOF1.5 (XSHUT)
- new net: JTOF1_1.5 (Pin_5), UTOF1.3 (GND)
- new net: JTOF1_1.6 (Pin_6), UTOF1.2 (VIN)
- new net TOF2_EXTI: JTOF1_0.3 (Pin_3)
- new net TOF2_SCL: JTOF1_0.2 (Pin_2), R302.1
- new net TOF2_SDA: JTOF1_0.1 (Pin_1), R301.1
- new net TOF2_XSHUT: JTOF1_0.4 (Pin_4)
- no-connect marks 1 -> 2
Other:
- note added: "VDD : Sortie regulateur 2.8 (utilisé en interne)"

Commit message: Update_Schemas
Parts:
- removed JCOLOR0: Conn_01x07_Female, Connector_JST:JST_XH_B7B-XH-AM_1x07_P2.50mm_Vertical, symbol Connector:Conn_01x07_Female
- removed JCOLOR1: Conn_01x07_Female, symbol Connector:Conn_01x07_Female
- removed JDistance0_2: Conn_01x03_Female, Connector_JST:JST_XH_B3B-XH-AM_1x03_P2.50mm_Vertical, symbol Connector:Conn_01x03_Female
- removed JDistance1_2: Conn_01x03_Female, symbol Connector:Conn_01x03_Female
- removed JTOF1_0: Conn_01x06_Female, Connector_JST:JST_XH_B6B-XH-AM_1x06_P2.50mm_Vertical, symbol Connector:Conn_01x06_Female
- removed JTOF1_1: Conn_01x06_Female, symbol Connector:Conn_01x06_Female
- removed R301, R302: 1k, Resistor_SMD:R_0603_1608Metric_Pad0.98x0.95mm_HandSolder, symbol Device:R_Small
- removed UDistance2: Distance-Sensor-GP2Y0D805Z0F, symbol Sensors_Beerator:Distance-Sensor-GP2Y0D805Z0F
- removed UTOF1: TOF-SENSOR-VL53LX, symbol Sensors_Beerator:TOF-SENSOR-VL53LX
- added JCOLOR_401, JCOLOR_403: Conn_01x05_Female, Connector_JST:JST_XH_B5B-XH-AM_1x05_P2.50mm_Vertical, symbol Connector:Conn_01x05_Female
- added JCOLOR_402, JCOLOR_404: Conn_01x05_Female, symbol Connector:Conn_01x05_Female
- added JDistance0_401: Conn_01x03_Female, Connector_JST:JST_XH_B3B-XH-AM_1x03_P2.50mm_Vertical, symbol Connector:Conn_01x03_Female
- added JDistance1_401: Conn_01x03_Female, symbol Connector:Conn_01x03_Female
- added JTOF1_401: Conn_01x06_Female, Connector_JST:JST_XH_B6B-XH-AM_1x06_P2.50mm_Vertical, symbol Connector:Conn_01x06_Female
- added JTOF1_403: Conn_01x06_Female, symbol Connector:Conn_01x06_Female
- added R401, R403: 1k, Resistor_SMD:R_0603_1608Metric_Pad0.98x0.95mm_HandSolder, symbol Device:R_Small
- added UDistance401: Distance-Sensor-GP2Y0D805Z0F, symbol Sensors_Beerator:Distance-Sensor-GP2Y0D805Z0F
- added UTOF401: TOF-SENSOR-VL53LX, symbol Sensors_Beerator:TOF-SENSOR-VL53LX
- renumbered JDistance0_1 to JDistance0_402, JDistance1_1 to JDistance1_402, JTOF0_0 to JTOF0_402, JTOF0_1 to JTOF0_404, R304 to R402, R303 to R404, UColor0 to UColor401, UDistance1 to UDistance402, UTOF0 to UTOF402
Connections:
- net GND: now also JDistance0_402.1 (Pin_1), JCOLOR_401.2 (Pin_2), JCOLOR_401.5 (Pin_5), JDistance0_401.1 (Pin_1), JTOF1_401.5 (Pin_5); no longer JDistance0_402.2 (Pin_2)
- net IR1-OUT: now also JDistance0_402.3 (Pin_3); no longer JDistance0_402.1 (Pin_1)
- net IR2-OUT: now also JDistance0_401.3 (Pin_3)
- net TCS-OUT: now also JCOLOR_404.5 (Pin_5)
- net TCS-S0: now also JCOLOR_404.1 (Pin_1)
- net TCS-S1: now also JCOLOR_404.2 (Pin_2)
- net TCS-S2: now also JCOLOR_404.3 (Pin_3)
- net TCS-S3: now also JCOLOR_404.4 (Pin_4)
- net TOF-EXTI: now also JTOF0_402.1 (Pin_1); no longer JTOF0_402.4 (Pin_4)
- net TOF-SCL: now also JTOF0_402.3 (Pin_3), R404.2; no longer JTOF0_402.2 (Pin_2), R402.1
- net TOF-SDA: now also JTOF0_402.4 (Pin_4), R402.1; no longer JTOF0_402.1 (Pin_1), R404.1
- net TOF-XSHUT: now also JTOF0_402.2 (Pin_2); no longer JTOF0_402.3 (Pin_3)
- net TOF2_EXTI: now also JTOF1_401.1 (Pin_1)
- net TOF2_SCL: now also JTOF1_401.3 (Pin_3), R403.1
- net TOF2_SDA: now also JTOF1_401.4 (Pin_4), R401.2
- net TOF2_XSHUT: now also JTOF1_401.2 (Pin_2)
- net at UDistance402.11 (Vin): now also JDistance1_402.2 (Pin_2); no longer JDistance1_402.3 (Pin_3)
- net at UDistance402.13 (OUT): now also JDistance1_402.3 (Pin_3); no longer JDistance1_402.1 (Pin_1)
- net at UDistance402.4 (GND): now also JDistance1_402.1 (Pin_1); no longer JDistance1_402.2 (Pin_2)
- net at UColor401.5 (VDD): now also JCOLOR_402.1 (Pin_1)
- net at UColor401.4 (GND): now also JCOLOR_402.2 (Pin_2)
- net at UColor401.1 (S0): now also JCOLOR_403.1 (Pin_1)
- net at UColor401.2 (S1): now also JCOLOR_403.2 (Pin_2)
- net at UColor401.7 (S2): now also JCOLOR_403.3 (Pin_3)
- net at UColor401.8 (S3): now also JCOLOR_403.4 (Pin_4)
- net at UColor401.6 (OUT): now also JCOLOR_403.5 (Pin_5)
- net at JTOF0_404.1 (Pin_1): now also UTOF402.7 (GPIO1); no longer UTOF402.9 (SDA)
- net at JTOF0_404.2 (Pin_2): now also UTOF402.5 (XSHUT); no longer UTOF402.7 (GPIO1)
- net at JTOF0_404.4 (Pin_4): now also UTOF402.9 (SDA); no longer UTOF402.5 (XSHUT)
- net 3.3 renamed +3.3V
- net +3.3V: now also JDistance0_402.2 (Pin_2), R404.1, JDistance0_401.2 (Pin_2), JTOF1_401.6 (Pin_6), R401.1, R403.2; no longer JDistance0_402.3 (Pin_3), R404.2
- new net: JDistance1_401.2 (Pin_2), UDistance401.11 (Vin)
- new net: JDistance1_401.3 (Pin_3), UDistance401.13 (OUT)
- new net: JDistance1_401.1 (Pin_1), UDistance401.4 (GND)
- new net: JTOF1_403.1 (Pin_1), UTOF401.7 (GPIO1)
- new net: JTOF1_403.2 (Pin_2), UTOF401.5 (XSHUT)
- new net: JTOF1_403.3 (Pin_3), UTOF401.10 (SCL)
- new net: JTOF1_403.4 (Pin_4), UTOF401.9 (SDA)
- new net: JTOF1_403.5 (Pin_5), UTOF401.3 (GND)
- new net: JTOF1_403.6 (Pin_6), UTOF401.2 (VIN)
- new net: JCOLOR_402.3 (Pin_3), UColor401. (OE)
- new net: JCOLOR_402.4 (Pin_4), UColor401. (OE)
- new net: JCOLOR_402.5 (Pin_5), UColor401. (OE)
- new net +5V: JCOLOR_401.1 (Pin_1)
- new net TCS-LED: JCOLOR_401.4 (Pin_4)
- new net TCS-OE: JCOLOR_401.3 (Pin_3)
Other:
- moved on the sheet: JTOF0_402, JTOF0_404, R402, R404, UTOF402

Commit message: pcb_v2
Parts:
- JCOLOR_403: footprint Connector_JST:JST_XH_B5B-XH-AM_1x05_P2.50mm_Vertical -> (none)
- JCOLOR_404: footprint (none) -> Connector_JST:JST_XH_B5B-XH-AM_1x05_P2.50mm_Vertical
Changed lines of the file:
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@@
     (property "Reference" "JCOLOR_404" (id 0) (at 125.73 49.53 0))
     (property "Value" "Conn_01x05_Female" (id 1) (at 125.73 52.07 0))
-    (property "Footprint" "" (id 2) (at 125.73 41.91 0)
+    (property "Footprint" "Connector_JST:JST_XH_B5B-XH-AM_1x05_P2.50mm_Vertical" (id 2) (at 125.73 41.91 0)
       (effects (font (size 1.27 1.27)) hide)
     )
@@
       (effects (font (size 1.27 1.27)) (justify left))
     )
-    (property "Footprint" "Connector_JST:JST_XH_B5B-XH-AM_1x05_P2.50mm_Vertical" (id 2) (at 111.76 41.91 0)
-      (effects (font (size 1.27 1.27)) hide)
-    )
+    (property "Footprint" "" (id 2) (at 111.76 41.91 0)
+      (effects (font (size 1.27 1.27)) hide)
+    )

Commit message: version_finale_pcb
Parts:
- renumbered JTOF0_402 to JTOF0_401, JTOF0_404 to JTOF0_402, JTOF1_403 to JTOF1_402
Changed lines of the file:
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@@
   (symbol (lib_id "Connector:Conn_01x06_Female") (at 236.22 48.26 180) (unit 1)
     (in_bom yes) (on_board yes)
-    (property "Reference" "JTOF0_404" (id 0) (at 245.11 34.29 0))
+    (property "Reference" "JTOF0_402" (id 0) (at 245.11 34.29 0))
     (property "Value" "Conn_01x06_Female" (id 1) (at 246.38 36.83 0))
     (property "Footprint" "" (id 2) (at 236.22 48.26 0)
@@
   (symbol (lib_id "Connector:Conn_01x06_Female") (at 234.95 115.57 180) (unit 1)
     (in_bom yes) (on_board yes)
-    (property "Reference" "JTOF1_403" (id 0) (at 243.84 101.6 0))
+    (property "Reference" "JTOF1_402" (id 0) (at 243.84 101.6 0))
     (property "Value" "Conn_01x06_Female" (id 1) (at 245.11 104.14 0))
     (property "Footprint" "" (id 2) (at 234.95 115.57 0)
@@
   (symbol (lib_id "Connector:Conn_01x06_Female") (at 223.52 50.8 0) (mirror x) (unit 1)
     (in_bom yes) (on_board yes)
-    (property "Reference" "JTOF0_402" (id 0) (at 217.17 34.29 0))
+    (property "Reference" "JTOF0_401" (id 0) (at 217.17 34.29 0))
     (property "Value" "Conn_01x06_Female" (id 1) (at 219.71 39.37 0))
     (property "Footprint" "Connector_JST:JST_XH_B6B-XH-AM_1x06_P2.50mm_Vertical" (id 2) (at 223.52 50.8 0)
