File: KiCad/Beerator/Beerator.kicad_pcb (KiCad board)
At the start: 2 copper layers, 24 parts

Commit message: feat(last pcb version)
Parts:
- removed C1: 10uF, Capacitor_SMD:C_0603_1608Metric_Pad1.08x0.95mm_HandSolder
- removed C2: 22uF, Capacitor_SMD:C_0603_1608Metric_Pad1.08x0.95mm_HandSolder
- removed C3, C4: 10u, Capacitor_SMD:C_0603_1608Metric_Pad1.08x0.95mm_HandSolder
- removed JDistance1_1: Conn_01x03_Female, Connector_JST:JST_EH_B3B-EH-A_1x03_P2.50mm_Vertical
- removed JTOF0: Conn_01x06_Female, Connector_JST:JST_EH_B6B-EH-A_1x06_P2.50mm_Vertical
- removed R1: 3meg, Resistor_SMD:R_0603_1608Metric_Pad0.98x0.95mm_HandSolder
- removed R2: 1,5meg, Resistor_SMD:R_0603_1608Metric_Pad0.98x0.95mm_HandSolder
- added C101: 10uF, Capacitor_SMD:C_0603_1608Metric_Pad1.08x0.95mm_HandSolder, F.Cu at (165.2, 103.6)
- added C102: 22uF, Capacitor_SMD:C_0603_1608Metric_Pad1.08x0.95mm_HandSolder, F.Cu at (165.0, 109.0)
- added C103: 1uF, Capacitor_SMD:C_0603_1608Metric_Pad1.08x0.95mm_HandSolder, F.Cu at (176.0, 109.0)
- added C104: 1uF, Capacitor_SMD:C_0603_1608Metric_Pad1.08x0.95mm_HandSolder, F.Cu at (168.0, 107.0)
- added C206: 100uF, Capacitor_THT:CP_Radial_D5.0mm_P2.00mm, F.Cu at (119.6, 73.6)
- added C207: 0.1uF, Capacitor_SMD:C_0603_1608Metric_Pad1.08x0.95mm_HandSolder, F.Cu at (190.0, 98.6)
- added C208: 0.1uF, Capacitor_SMD:C_0603_1608Metric_Pad1.08x0.95mm_HandSolder, F.Cu at (190.0, 92.8)
- added C209: 0.1uF, Capacitor_SMD:C_0603_1608Metric_Pad1.08x0.95mm_HandSolder, F.Cu at (95.1, 95.3)
- added C210: 0.1uF, Capacitor_SMD:C_0603_1608Metric_Pad1.08x0.95mm_HandSolder, F.Cu at (95.1, 98.3)
- added C401: 15p, Capacitor_SMD:C_0603_1608Metric_Pad1.08x0.95mm_HandSolder, F.Cu at (127.8, 98.6)
- added C402: 15p, Capacitor_SMD:C_0603_1608Metric_Pad1.08x0.95mm_HandSolder, F.Cu at (132.2, 104.2)
- added C403: 100n, Capacitor_SMD:C_0603_1608Metric_Pad1.08x0.95mm_HandSolder, F.Cu at (125.8, 98.8)
- added C404: 4,7u, Capacitor_THT:CP_Radial_D5.0mm_P2.00mm, F.Cu at (121.6, 98.0)
- added D101: LED_Small, LED_SMD:LED_0603_1608Metric_Pad1.05x0.95mm_HandSolder, F.Cu at (149.0, 99.0)
- added D102: LED_Small, LED_SMD:LED_0603_1608Metric_Pad1.05x0.95mm_HandSolder, F.Cu at (180.0, 111.0)
- added H101: MountingHole_Pad, MountingHole:MountingHole_3.2mm_M3_Pad_Via, F.Cu at (192.0, 107.0)
- added H102: MountingHole_Pad, MountingHole:MountingHole_3.2mm_M3_Pad_Via, F.Cu at (92.0, 107.0)
- added H103: MountingHole_Pad, MountingHole:MountingHole_3.2mm_M3_Pad_Via, F.Cu at (192.0, 67.0)
- added H104: MountingHole_Pad, MountingHole:MountingHole_3.2mm_M3_Pad_Via, F.Cu at (92.0, 67.0)
- added JDistance0_2: Conn_01x03_Female, Connector_JST:JST_XH_B3B-XH-AM_1x03_P2.50mm_Vertical, F.Cu at (186.0, 74.7)
- added JP1: SolderJumper_2_Open, Jumper:SolderJumper-3_P2.0mm_Open_TrianglePad1.0x1.5mm, F.Cu at (149.4, 81.6)
- added JP2: SolderJumper_2_Open, Jumper:SolderJumper-3_P2.0mm_Open_TrianglePad1.0x1.5mm, F.Cu at (149.6, 85.0)
- added JP3: SolderJumper_2_Open, Jumper:SolderJumper-3_P2.0mm_Open_TrianglePad1.0x1.5mm, F.Cu at (101.6, 98.0)
- added JP4: SolderJumper_2_Open, Jumper:SolderJumper-3_P2.0mm_Open_TrianglePad1.0x1.5mm, F.Cu at (98.6, 94.4)
- added JP5: SolderJumper_2_Open, Jumper:SolderJumper-3_P2.0mm_Open_TrianglePad1.0x1.5mm, F.Cu at (185.4, 99.0)
- added JP6: SolderJumper_2_Open, Jumper:SolderJumper-3_P2.0mm_Open_TrianglePad1.0x1.5mm, F.Cu at (182.2, 103.4)
- added JSTLINK1: Conn_02x07_Odd_Even, Connector_PinHeader_1.27mm:PinHeader_2x07_P1.27mm_Vertical_SMD, F.Cu at (161.6, 81.2)
- added JTOF0_0: Conn_01x06_Female, Connector_JST:JST_XH_B6B-XH-AM_1x06_P2.50mm_Vertical, F.Cu at (163.8, 65.7)
- added JTOF1_0: Conn_01x06_Female, Connector_JST:JST_XH_B6B-XH-AM_1x06_P2.50mm_Vertical, F.Cu at (113.6, 65.8)
- added R103: 215, Resistor_SMD:R_0603_1608Metric_Pad0.98x0.95mm_HandSolder, F.Cu at (149.0, 101.0)
- added R105: 215, Resistor_SMD:R_0603_1608Metric_Pad0.98x0.95mm_HandSolder, F.Cu at (180.0, 109.0)
- added R205: 10k, Resistor_SMD:R_0603_1608Metric_Pad0.98x0.95mm_HandSolder, F.Cu at (123.4, 71.6)
- added R301: 1k, Resistor_SMD:R_0603_1608Metric_Pad0.98x0.95mm_HandSolder, F.Cu at (117.8, 65.0)
- added R302: 1k, Resistor_SMD:R_0603_1608Metric_Pad0.98x0.95mm_HandSolder, F.Cu at (96.6, 64.2)
- added R303: 1k, Resistor_SMD:R_0603_1608Metric_Pad0.98x0.95mm_HandSolder, F.Cu at (159.8, 65.8)
- added R304: 1k, Resistor_SMD:R_0603_1608Metric_Pad0.98x0.95mm_HandSolder, F.Cu at (182.9, 64.2)
- added R401: 80, Resistor_SMD:R_0603_1608Metric_Pad0.98x0.95mm_HandSolder, F.Cu at (129.6, 98.6)
- added SW1: SW_DPDT_x2, SamacSys_Parts:NE555DR, F.Cu at (150.0, 108.0)
- added Y401: 16MHz, Crystal:Crystal_SMD_0603-4Pin_6.0x3.5mm, F.Cu at (127.2, 104.2)
- C201, C202: footprint Capacitor_SMD:C_0603_1608Metric_Pad1.08x0.95mm_HandSolder -> Capacitor_THT:CP_Radial_D5.0mm_P2.00mm
- C204, C205: value 10µF -> 1µF
- JCOLOR0: footprint Connector_JST:JST_EH_B7B-EH-A_1x07_P2.50mm_Vertical -> Connector_JST:JST_XH_B7B-XH-AM_1x07_P2.50mm_Vertical
- JDistance0_1: footprint Connector_JST:JST_EH_B3B-EH-A_1x03_P2.50mm_Vertical -> Connector_JST:JST_XH_B3B-XH-AM_1x03_P2.50mm_Vertical
- JMCC1_0, JMCC2_0: footprint Connector_JST:JST_EH_B6B-EH-A_1x06_P2.50mm_Vertical -> Connector_JST:JST_XH_B6B-XH-AM_1x06_P2.50mm_Vertical
- JSERVO0: footprint Connector_JST:JST_XA_B03B-XASK-1-A_1x03_P2.50mm_Vertical -> Connector_JST:JST_XH_B3B-XH-AM_1x03_P2.50mm_Vertical
- moved REG3-3 131.6 mm to (172.0, 109.0)
- moved C202 131.4 mm to (183.2, 84.0), turned to 90 degrees
- moved C204 117.1 mm to (176.0, 90.0)
- moved JBat1 90.2 mm to (140.6, 107.0)
- moved REG5 87.5 mm to (159.0, 108.0), turned to 180 degrees
- moved JMCC2_0 80.6 mm to (195.1, 85.5)
- moved UDRIVER2 76.5 mm to (182.4, 90.2), turned to -90 degrees
- moved JCOLOR0 62.0 mm to (137.0, 65.7), turned to 0 degrees
- moved USTM1 59.5 mm to (128.0, 88.4), turned to 90 degrees
- moved C201 58.6 mm to (103.0, 81.2)
- moved UDRIVER1 56.8 mm to (102.8, 88.2), turned to -90 degrees
- moved JMCC1_0 56.6 mm to (90.1, 85.3), turned to -90 degrees
- moved C203 54.7 mm to (118.6, 69.6)
- moved C205 51.8 mm to (96.4, 89.2), turned to 90 degrees
- moved JDistance0_1 48.0 mm to (92.5, 75.7)
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Connections:
- C201 pad 1: Net-(C201-Pad1) -> 7.2
- C201 pad 2: 7.2 -> GND
- C202 pad 1: Net-(C202-Pad1) -> 7.2
- C202 pad 2: 7.2 -> GND
- C203 pad 1: 7.2 -> GND
- C204 pad 1: 7.2 -> GND
- C204 pad 2: 7.2 -> 5
- C205 pad 1: 7.2 -> GND
- C205 pad 2: 7.2 -> 5
- JBat1 pad 1: 7.2 -> GND
- JBat1 pad 2: 7.2 -> Net-(JBat1-Pad2)
- JCOLOR0 pad 2: 7.2 -> GND
- JDistance0_1 pad 2: 7.2 -> GND
- JMCC1_0 pad 3: 7.2 -> GND
- JMCC1_0 pad 5: 02_D1 -> O2_D1
- JMCC1_0 pad 6: 01_D1 -> O1_D1
- JMCC2_0 pad 1: PHASE_B_M2 -> PHASE_A_M2
- JMCC2_0 pad 2: PHASE_A_M2 -> PHASE_B_M2
- JMCC2_0 pad 3: 7.2 -> GND
- JMCC2_0 pad 5: 02_D2 -> O1_D2
- JMCC2_0 pad 6: 01_D2 -> O2_D2
- JSERVO0 pad 1: 7.2 -> GND
- REG3-3 pad 2: 7.2 -> GND
- REG3-3 pad 3: Net-(R1-Pad2) -> 5
- REG5 pad 1: 7.2 -> GND
- UDRIVER1 pad 1: O1_D1 -> Net-(JP3-Pad1)
- UDRIVER1 pad 2: Net-(C201-Pad1) -> 7.2
- UDRIVER1 pad 3: 7.2 -> 5
- UDRIVER1 pad 6: 7.2 -> GND
- UDRIVER1 pad 7: O2_D1 -> Net-(JP4-Pad1)
- UDRIVER1 pad 8: 7.2 -> GND
- UDRIVER2 pad 1: 01_D2 -> Net-(JP5-Pad1)
- UDRIVER2 pad 2: Net-(C202-Pad1) -> 7.2
- UDRIVER2 pad 3: 7.2 -> 5
- UDRIVER2 pad 6: 7.2 -> GND
- UDRIVER2 pad 7: 02_D2 -> Net-(JP6-Pad1)
- UDRIVER2 pad 8: 7.2 -> GND
- USTM1 pad 10: unconnected-(USTM1-Pad10) -> Net-(C401-Pad1)
- USTM1 pad 11: unconnected-(USTM1-Pad11) -> Net-(R401-Pad2)
- USTM1 pad 12: unconnected-(USTM1-Pad12) -> NRST
- USTM1 pad 18: unconnected-(USTM1-Pad18) -> NPWM_D2
- USTM1 pad 19: unconnected-(USTM1-Pad19) -> PWM_D2
- USTM1 pad 23: unconnected-(USTM1-Pad23) -> PWM_D1
- USTM1 pad 24: unconnected-(USTM1-Pad24) -> TCS-OUT
- USTM1 pad 25: unconnected-(USTM1-Pad25) -> TX
- USTM1 pad 26: unconnected-(USTM1-Pad26) -> RX
- USTM1 pad 28: unconnected-(USTM1-Pad28) -> TOF-EXTI
- USTM1 pad 29: unconnected-(USTM1-Pad29) -> TOF-XSHUT
- USTM1 pad 30: unconnected-(USTM1-Pad30) -> TOF-SCL
- USTM1 pad 31: unconnected-(USTM1-Pad31) -> TOF-SDA
- USTM1 pad 34: unconnected-(USTM1-Pad34) -> TCS-S3
- USTM1 pad 35: unconnected-(USTM1-Pad35) -> TCS-S2
- USTM1 pad 36: unconnected-(USTM1-Pad36) -> TCS-S1
- USTM1 pad 37: unconnected-(USTM1-Pad37) -> TCS-S0
- USTM1 pad 38: unconnected-(USTM1-Pad38) -> PHASE_B_M2
- USTM1 pad 39: unconnected-(USTM1-Pad39) -> PHASE_A_M2
- USTM1 pad 40: unconnected-(USTM1-Pad40) -> IR2-OUT
- USTM1 pad 41: unconnected-(USTM1-Pad41) -> IR1-OUT
- USTM1 pad 45: unconnected-(USTM1-Pad45) -> SWDIO
- USTM1 pad 46: unconnected-(USTM1-Pad46) -> SWCLK
- USTM1 pad 48: unconnected-(USTM1-Pad48) -> PHASE_B_M1
- USTM1 pad 49: unconnected-(USTM1-Pad49) -> PHASE_A_M1
- USTM1 pad 55: unconnected-(USTM1-Pad55) -> SERVO_DATA
- USTM1 pad 6: unconnected-(USTM1-Pad6) -> 3.3
- USTM1 pad 60: unconnected-(USTM1-Pad60) -> NPWM_D1
- USTM1 pad 61: unconnected-(USTM1-Pad61) -> TOF2_SDA
- USTM1 pad 62: unconnected-(USTM1-Pad62) -> TOF2_SCL
- USTM1 pad 63: unconnected-(USTM1-Pad63) -> TOF2_EXTI
- USTM1 pad 64: unconnected-(USTM1-Pad64) -> TOF2_XSHUT
- USTM1 pad 8: unconnected-(USTM1-Pad8) -> Net-(C403-Pad2)
- USTM1 pad 9: unconnected-(USTM1-Pad9) -> GND
Routing:
- net 3.3: track 0.00 -> 277.2 mm, vias 0 -> 3
- net 7.2: track 0.00 -> 172.2 mm, vias 0 -> 2
- net 5: track 0.00 -> 114.0 mm
- net PHASE_A_M2: track 0.00 -> 81.6 mm, vias 0 -> 2
- net PHASE_B_M2: track 0.00 -> 80.7 mm, vias 0 -> 2
- net IR2-OUT: track 0.00 -> 70.7 mm, vias 0 -> 2
- net SWDIO: track 0.00 -> 64.8 mm, vias 0 -> 2
- net SWCLK: track 0.00 -> 63.4 mm, vias 0 -> 2
- net TOF-SCL: track 0.00 -> 58.7 mm
- net PHASE_B_M1: track 0.00 -> 56.3 mm, vias 0 -> 2
- net NPWM_D2: track 0.00 -> 52.5 mm, vias 0 -> 2
- net PWM_D2: track 0.00 -> 51.2 mm, vias 0 -> 2
- net PHASE_A_M1: track 0.00 -> 50.6 mm, vias 0 -> 2
- net PWM_D1: track 0.00 -> 49.9 mm, vias 0 -> 2
- net IR1-OUT: track 0.00 -> 48.8 mm, vias 0 -> 2
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- added copper zone on In2.Cu, net 5
- added copper zone on B.Cu, net GND
- added copper zone on F.Cu, net GND
- added copper zone on In1.Cu, net GND
Other:
- board outline added: 112 x 52 mm
- copper layers 2 -> 4

Commit message: pcb_v2
Parts:
- removed C101: 10uF, Capacitor_SMD:C_0603_1608Metric_Pad1.08x0.95mm_HandSolder
- removed C102: 22uF, Capacitor_SMD:C_0603_1608Metric_Pad1.08x0.95mm_HandSolder
- removed C103, C104: 1uF, Capacitor_SMD:C_0603_1608Metric_Pad1.08x0.95mm_HandSolder
- removed C205: 1µF, Capacitor_SMD:C_0603_1608Metric_Pad1.08x0.95mm_HandSolder
- removed C206: 100uF, Capacitor_THT:CP_Radial_D5.0mm_P2.00mm
- removed C207, C208, C209, C210: 0.1uF, Capacitor_SMD:C_0603_1608Metric_Pad1.08x0.95mm_HandSolder
- removed C401, C402: 15p, Capacitor_SMD:C_0603_1608Metric_Pad1.08x0.95mm_HandSolder
- removed C403: 100n, Capacitor_SMD:C_0603_1608Metric_Pad1.08x0.95mm_HandSolder
- removed C404: 4,7u, Capacitor_THT:CP_Radial_D5.0mm_P2.00mm
- removed D101, D102: LED_Small, LED_SMD:LED_0603_1608Metric_Pad1.05x0.95mm_HandSolder
- removed JBat1: Conn_01x02_Female, Connector_JST:JST_XH_B2B-XH-AM_1x02_P2.50mm_Vertical
- removed JCOLOR0: Conn_01x07_Female, Connector_JST:JST_XH_B7B-XH-AM_1x07_P2.50mm_Vertical
- removed JDistance0_1, JDistance0_2, JSERVO0: Conn_01x03_Female, Connector_JST:JST_XH_B3B-XH-AM_1x03_P2.50mm_Vertical
- removed JMCC1_0, JMCC2_0, JTOF0_0, JTOF1_0: Conn_01x06_Female, Connector_JST:JST_XH_B6B-XH-AM_1x06_P2.50mm_Vertical
- removed JP1, JP2, JP3, JP4, JP5, JP6: SolderJumper_2_Open, Jumper:SolderJumper-3_P2.0mm_Open_TrianglePad1.0x1.5mm
- removed JSTLINK1: Conn_02x07_Odd_Even, Connector_PinHeader_1.27mm:PinHeader_2x07_P1.27mm_Vertical_SMD
- removed R103, R105: 215, Resistor_SMD:R_0603_1608Metric_Pad0.98x0.95mm_HandSolder
- removed R205: 10k, Resistor_SMD:R_0603_1608Metric_Pad0.98x0.95mm_HandSolder
- removed R302, R303, R304: 1k, Resistor_SMD:R_0603_1608Metric_Pad0.98x0.95mm_HandSolder
- removed REG3-3: MCP1802x-xx02xOT, Package_TO_SOT_SMD:SOT-23-5
- removed REG5: AZ1117-5.0, Package_TO_SOT_SMD:SOT-223
- removed SW1: SW_DPDT_x2, SamacSys_Parts:NE555DR
- removed UDRIVER1, UDRIVER2: ZXBM5210-S, Package_SO:SOIC-8_3.9x4.9mm_P1.27mm
- removed USTM1: STM32G070RBT6, Package_QFP:LQFP-64-1EP_10x10mm_P0.5mm_EP6.5x6.5mm
- removed Y401: 16MHz, Crystal:Crystal_SMD_0603-4Pin_6.0x3.5mm
- added C301: 4,7u, Capacitor_THT:CP_Radial_D5.0mm_P2.00mm, F.Cu at (83.8, 65.8)
- added C302: 15p, Capacitor_SMD:C_0603_1608Metric_Pad1.08x0.95mm_HandSolder, F.Cu at (87.6, 69.6)
- added C303: 15p, Capacitor_SMD:C_0603_1608Metric_Pad1.08x0.95mm_HandSolder, F.Cu at (87.6, 74.6)
- added C304: 100n, Capacitor_SMD:C_0603_1608Metric_Pad1.08x0.95mm_HandSolder, F.Cu at (89.2, 68.0)
- added C501: 1µF, Capacitor_SMD:C_0603_1608Metric_Pad1.08x0.95mm_HandSolder, F.Cu at (64.4, 67.8)
- added C502: 1µF, Capacitor_SMD:C_0603_1608Metric_Pad1.08x0.95mm_HandSolder, F.Cu at (138.2, 80.4)
- added C503: 10µF, Capacitor_THT:CP_Radial_D5.0mm_P2.00mm, F.Cu at (71.4, 66.0)
- added C504: 10µF, Capacitor_THT:CP_Radial_D5.0mm_P2.00mm, F.Cu at (131.2, 82.0)
- added C505: 100uF, Capacitor_THT:CP_Radial_D5.0mm_P2.00mm, F.Cu at (93.8, 56.8)
- added C506: 0.1uF, Capacitor_SMD:C_0603_1608Metric_Pad1.08x0.95mm_HandSolder, F.Cu at (144.2, 67.4)
- added C507: 0.1uF, Capacitor_SMD:C_0603_1608Metric_Pad1.08x0.95mm_HandSolder, F.Cu at (100.0, 55.6)
- added C508: 0.1uF, Capacitor_SMD:C_0603_1608Metric_Pad1.08x0.95mm_HandSolder, F.Cu at (56.0, 78.8)
- added C509: 0.1uF, Capacitor_SMD:C_0603_1608Metric_Pad1.08x0.95mm_HandSolder, F.Cu at (143.3, 80.8)
- added C510: 0.1uF, Capacitor_SMD:C_0603_1608Metric_Pad1.08x0.95mm_HandSolder, F.Cu at (56.0, 66.0)
- added D201: LED_Small, LED_SMD:LED_0603_1608Metric_Pad1.05x0.95mm_HandSolder, F.Cu at (109.8, 82.2)
- added D202: LED_Small, LED_SMD:LED_0603_1608Metric_Pad1.05x0.95mm_HandSolder, F.Cu at (116.2, 80.4)
- added JBat201: Conn_01x02_Female, Connector_JST:JST_XH_B2B-XH-AM_1x02_P2.50mm_Vertical, F.Cu at (98.8, 91.7)
- added JCOLOR_401: Conn_01x05_Female, Connector_JST:JST_XH_B5B-XH-AM_1x05_P2.50mm_Vertical, F.Cu at (79.2, 48.7)
- added JCOLOR_404: Conn_01x05_Female, Connector_JST:JST_XH_B5B-XH-AM_1x05_P2.50mm_Vertical, F.Cu at (109.8, 48.9)
- added JDistance0_401: Conn_01x03_Female, Connector_JST:JST_XH_B3B-XH-AM_1x03_P2.50mm_Vertical, F.Cu at (70.4, 91.8)
- added JDistance0_402: Conn_01x03_Female, Connector_JST:JST_XH_B3B-XH-AM_1x03_P2.50mm_Vertical, F.Cu at (84.1, 91.7)
- added JMCC0_502: Conn_01x06_Female, Connector_JST:JST_XH_B6B-XH-AM_1x06_P2.50mm_Vertical, F.Cu at (48.9, 66.2)
- added JMCC1_501: Conn_01x06_Female, Connector_JST:JST_XH_B6B-XH-AM_1x06_P2.50mm_Vertical, F.Cu at (150.9, 80.2)
- added JP301: SolderJumper_2_Open, Jumper:SolderJumper-3_P2.0mm_Open_TrianglePad1.0x1.5mm, F.Cu at (119.0, 65.0)
- added JP302: SolderJumper_2_Open, Jumper:SolderJumper-3_P2.0mm_Open_TrianglePad1.0x1.5mm, F.Cu at (120.8, 68.4)
- added JP501: SolderJumper_2_Open, Jumper:SolderJumper-3_P2.0mm_Open_TrianglePad1.0x1.5mm, F.Cu at (55.0, 63.8)
- added JP502: SolderJumper_2_Open, Jumper:SolderJumper-3_P2.0mm_Open_TrianglePad1.0x1.5mm, F.Cu at (55.2, 81.4)
- added JP503: SolderJumper_2_Open, Jumper:SolderJumper-3_P2.0mm_Open_TrianglePad1.0x1.5mm, F.Cu at (144.2, 83.0)
- added JP504: SolderJumper_2_Open, Jumper:SolderJumper-3_P2.0mm_Open_TrianglePad1.0x1.5mm, F.Cu at (145.0, 65.0)
- added JSERVO501: Conn_01x03_Female, Connector_JST:JST_XH_B3B-XH-AM_1x03_P2.50mm_Vertical, F.Cu at (101.8, 49.6)
- added JSTLINK301: Conn_02x07_Odd_Even, Connector_PinHeader_1.27mm:PinHeader_2x07_P1.27mm_Vertical_SMD, F.Cu at (111.0, 65.4)
- added JTOF0_402: Conn_01x06_Female, Connector_JST:JST_XH_B6B-XH-AM_1x06_P2.50mm_Vertical, F.Cu at (139.8, 48.8)
- added JTOF1_401: Conn_01x06_Female, Connector_JST:JST_XH_B6B-XH-AM_1x06_P2.50mm_Vertical, F.Cu at (59.0, 48.7)
- added R201: 4,2k, Resistor_SMD:R_0603_1608Metric_Pad0.98x0.95mm_HandSolder, F.Cu at (111.6, 84.0)
- added R202: 300, Resistor_SMD:R_0603_1608Metric_Pad0.98x0.95mm_HandSolder, F.Cu at (117.8, 80.4)
- added R402: 1k, Resistor_SMD:R_0603_1608Metric_Pad0.98x0.95mm_HandSolder, F.Cu at (133.4, 54.8)
- added R403: 1k, Resistor_SMD:R_0603_1608Metric_Pad0.98x0.95mm_HandSolder, F.Cu at (64.2, 55.0)
- added R404: 1k, Resistor_SMD:R_0603_1608Metric_Pad0.98x0.95mm_HandSolder, F.Cu at (135.2, 54.8)
- added R501: 10k, Resistor_SMD:R_0603_1608Metric_Pad0.98x0.95mm_HandSolder, F.Cu at (104.2, 54.0)
- added REG201: AZ1117-5.0, Package_TO_SOT_SMD:SOT-223, F.Cu at (115.4, 90.6)
- added REG3-201: MCP1802x-xx02xOT, Package_TO_SOT_SMD:SOT-23-5, F.Cu at (121.2, 83.2)
- added SW201: SW_DPDT_x2, SamacSys_Parts:NE555DR, F.Cu at (107.6, 91.6)
- added UDRIVER501: ZXBM5210-S, Package_SO:SOIC-8_3.9x4.9mm_P1.27mm, F.Cu at (65.8, 73.0)
- added UDRIVER502: ZXBM5210-S, Package_SO:SOIC-8_3.9x4.9mm_P1.27mm, F.Cu at (136.4, 75.4)
- added USTM301: STM32G070RBT6, Package_QFP:LQFP-64_10x10mm_P0.5mm, F.Cu at (97.6, 70.4)
- added Y301: 16MHz, Crystal:Crystal_SMD_0603-4Pin_6.0x3.5mm, F.Cu at (84.0, 73.6)
- C201: value 10µF -> 10uF; footprint Capacitor_THT:CP_Radial_D5.0mm_P2.00mm -> Capacitor_SMD:C_0603_1608Metric_Pad1.08x0.95mm_HandSolder
- C202: value 10µF -> 22uF; footprint Capacitor_THT:CP_Radial_D5.0mm_P2.00mm -> Capacitor_SMD:C_0603_1608Metric_Pad1.08x0.95mm_HandSolder
- C203: value 0.1uF -> 1uF
- C204: value 1µF -> 1uF
- R301: value 1k -> 80
- R401: value 80 -> 1k
- moved H101 153.0 mm to (50.0, 50.0), turned to 0 degrees
- moved H103 143.9 mm to (50.0, 90.0), turned to 0 degrees
- moved H102 81.3 mm to (150.0, 50.0), turned to 0 degrees
- moved R401 77.3 mm to (65.8, 55.0)
- moved C202 67.8 mm to (115.4, 84.0)
- moved H104 62.4 mm to (150.0, 90.0), turned to 0 degrees
- moved C204 55.7 mm to (121.2, 80.2)
- moved R301 30.1 mm to (88.6, 72.2), turned to 0 degrees
- moved C203 14.4 mm to (118.0, 84.0), turned to 90 degrees
- moved C201 10.5 mm to (113.2, 84.0), turned to 90 degrees
Connections:
- C201 pad 1: 7.2 -> +BATT
- C202 pad 1: 7.2 -> +5V
- C203 pad 1: GND -> +5V
- C203 pad 2: 7.2 -> GND
- C204 pad 1: GND -> +3.3V
- C204 pad 2: 5 -> GND
- R301 pad 1: TOF2_SDA -> Net-(C303-Pad2)
- R301 pad 2: 3.3 -> Net-(R301-Pad2)
- R401 pad 1: Net-(C402-Pad2) -> +3.3V
- R401 pad 2: Net-(R401-Pad2) -> TOF2_SDA
Routing:
- net 3.3: track 277.2 -> 0.00 mm, vias 3 -> 0
- net +5V: track 0.00 -> 196.9 mm, vias 0 -> 4
- net 7.2: track 172.2 -> 0.00 mm, vias 2 -> 0
- net +BATT: track 0.00 -> 143.5 mm
- net 5: track 114.0 -> 0.00 mm
- net SWDIO: track 64.8 -> 5.87 mm, vias 2 -> 0
- net SWCLK: track 63.4 -> 6.19 mm, vias 2 -> 0
- net IR2-OUT: track 70.7 -> 27.3 mm, vias 2 -> 1
- net +3.3V: track 0.00 -> 43.3 mm, vias 0 -> 2
- net PHASE_A_M2: track 81.6 -> 50.2 mm, vias 2 -> 1
- net IR1-OUT: track 48.8 -> 18.4 mm, vias 2 -> 1
- net PHASE_B_M2: track 80.7 -> 51.6 mm, vias 2 -> 1
- net NPWM_D1: track 27.6 -> 55.1 mm
- net TCS-LED: track 0.00 -> 27.0 mm, vias 0 -> 1
- net TCS-OE: track 0.00 -> 26.6 mm, vias 0 -> 1
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- added copper zone on In2.Cu, net +3.3V
- removed copper zone on In2.Cu, net 5

Commit message: version_finale_pcb
Parts:
- removed REG201: AZ1117-5.0, Package_TO_SOT_SMD:SOT-223
- added U201: REG-5, Package_TO_SOT_SMD:SOT-223, F.Cu at (116.6, 87.8)
- JP301, JP302, JP501, JP502, JP503, JP504: footprint Jumper:SolderJumper-3_P2.0mm_Open_TrianglePad1.0x1.5mm -> Jumper:SolderJumper-2_P1.3mm_Open_Pad1.0x1.5mm
- Y301: value 16MHz -> Crystal_GND23; footprint Crystal:Crystal_SMD_0603-4Pin_6.0x3.5mm -> Crystal:Crystal_SMD_EuroQuartz_MT-4Pin_3.2x2.5mm
- moved C504 17.6 mm to (139.5, 66.5), turned to 0 degrees
- moved JP504 14.9 mm to (138.4, 78.4)
- moved JMCC1_501 14.9 mm to (149.2, 65.5), turned to -90 degrees
- moved C506 14.4 mm to (138.4, 80.6)
- moved JP302 14.3 mm to (109.8, 59.2), turned to 0 degrees
- moved C502 13.5 mm to (136.1, 67.1), turned to -90 degrees
- moved JP503 11.8 mm to (141.0, 71.6), turned to -90 degrees
- moved JP502 10.2 mm to (65.0, 78.4)
- moved C501 8.09 mm to (59.2, 74.0), turned to 90 degrees
- moved C503 7.85 mm to (63.6, 64.8), turned to 0 degrees
- moved C509 7.80 mm to (143.2, 73.0), turned to 90 degrees
- moved JP501 7.05 mm to (59.0, 69.6), turned to 90 degrees
- moved JDistance0_401 5.60 mm to (74.9, 88.5)
- moved JMCC0_501 4.88 mm to (53.8, 66.3)
- moved JDistance0_402 4.12 mm to (86.7, 88.5)
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- renumbered JMCC0_502 to JMCC0_501, JTOF0_402 to JTOF0_401
Connections:
- net Net-(JP301-Pad2) renamed /Control/RX_JP
- net Net-(JP302-Pad1) renamed /Control/TX_JP
- R501 pad 2: +5V -> +3.3V
- USTM301 pad 36: PHASE_B_M2 -> PHASE_A_M2
- USTM301 pad 37: PHASE_A_M2 -> PHASE_B_M2
- Y301 pad 2: Net-(C302-Pad1) -> GND
- Y301 pad 3: (no net) -> Net-(C302-Pad1)
- Y301 pad 4: (no net) -> GND
Routing:
- net +5V: track 196.9 -> 15.9 mm, vias 4 -> 1
- net +BATT: track 143.5 -> 277.4 mm
- net GND: track 5.13 -> 96.1 mm, vias 5 -> 10
- net Net-(JP501-Pad1): track 20.1 -> 2.63 mm
- net /Control/TX_JP: track 19.1 -> 2.43 mm
- net TX: track 18.5 -> 32.7 mm
- net Net-(JP503-Pad1): track 15.7 -> 2.24 mm
- net NPWM_D2: track 45.6 -> 33.4 mm, vias 2 -> 0
- net Net-(JP504-Pad1): track 12.8 -> 2.69 mm
- net PWM_D2: track 42.1 -> 32.7 mm, vias 2 -> 0
- net PWM_D1: track 49.9 -> 57.0 mm, vias 2 -> 0
- net NPWM_D1: track 55.1 -> 48.6 mm, vias 2 -> 0
- net IR2-OUT: track 27.3 -> 21.6 mm, vias 1 -> 0
- net TCS-S3: track 30.2 -> 24.8 mm, vias 0 -> 1
- net PHASE_B_M2: track 51.6 -> 46.6 mm
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- added copper zone on F.Cu, net +5V
- removed copper zone on F.Cu, net GND

Commit message: fichier_production
Other:
- board text added: "Beerator A.P"
Changed lines of the file:
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@@
       (outputformat 1)
       (mirror false)
-      (drillshape 1)
+      (drillshape 0)
       (scaleselection 1)
-      (outputdirectory "")
+      (outputdirectory "../../PCB_GERBER/")
     )
   )
@@
     (fp_line (start 14.95 3.4) (end 14.95 -2.35) (layer "F.Fab") (width 0.1))
     (pad "" np_thru_hole circle (at -1.6 2 270) (size 1.2 1.2) (drill 1.2) (layers *.Cu *.Mask))
-    (pad "1" thru_hole roundrect (at 0 0 270) (size 1.7 1.95) (drill 0.95) (layers *.Cu *.Mask) (roundrect_rratio 0.147059)
+    (pad "1" thru_hole roundrect (at 0 0 270) (size 1.7 1.95) (drill 0.95) (layers *.Cu *.Mask) (roundrect_rratio 0.1470588235)
       (net 7 "O1_D1") (pinfunction "Pin_1") (pintype "passive"))
     (pad "2" thru_hole oval (at 2.5 0 270) (size 1.7 1.95) (drill 0.95) (layers *.Cu *.Mask)
@@
     (fp_line (start 7.45 -2.35) (end -2.45 -2.35) (layer "F.Fab") (width 0.1))
     (pad "" np_thru_hole circle (at -1.6 2 180) (size 1.2 1.2) (drill 1.2) (layers *.Cu *.Mask))
-    (pad "1" thru_hole roundrect (at 0 0 180) (size 1.7 1.95) (drill 0.95) (layers *.Cu *.Mask) (roundrect_rratio 0.147059)
+    (pad "1" thru_hole roundrect (at 0 0 180) (size 1.7 1.95) (drill 0.95) (layers *.Cu *.Mask) (roundrect_rratio 0.1470588235)
       (net 29 "SERVO_DATA") (pinfunction "Pin_1") (pintype "passive"))
     (pad "2" thru_hole oval (at 2.5 0 180) (size 1.7 1.95) (drill 0.95) (layers *.Cu *.Mask)
@@
     (fp_line (start 14.95 -2.35) (end -2.45 -2.35) (layer "F.Fab") (width 0.1))
     (pad "" np_thru_hole circle (at -1.6 2 180) (size 1.2 1.2) (drill 1.2) (layers *.Cu *.Mask))
-    (pad "1" thru_hole roundrect (at 0 0 180) (size 1.7 1.95) (drill 0.95) (layers *.Cu *.Mask) (roundrect_rratio 0.147059)
+    (pad "1" thru_hole roundrect (at 0 0 180) (size 1.7 1.95) (drill 0.95) (layers *.Cu *.Mask) (roundrect_rratio 0.1470588235)
       (net 37 "TOF-EXTI") (pinfunction "Pin_1") (pintype "passive"))
     (pad "2" thru_hole oval (at 2.5 0 180) (size 1.7 1.95) (drill 0.95) (layers *.Cu *.Mask)
@@
     (fp_line (start -2.45 -2.35) (end -2.45 3.4) (layer "F.Fab") (width 0.1))
     (pad "" np_thru_hole circle (at -1.6 2) (size 1.2 1.2) (drill 1.2) (layers *.Cu *.Mask))
-    (pad "1" thru_hole roundrect (at 0 0) (size 1.7 1.95) (drill 0.95) (layers *.Cu *.Mask) (roundrect_rratio 0.147059)
+    (pad "1" thru_hole roundrect (at 0 0) (size 1.7 1.95) (drill 0.95) (layers *.Cu *.Mask) (roundrect_rratio 0.1470588235)
       (net 13 "TCS-S0") (pinfunction "Pin_1") (pintype "passive"))
     (pad "2" thru_hole oval (at 2.5 0) (size 1.7 1.95) (drill 0.95) (layers *.Cu *.Mask)
@@
     (fp_line (start 0 -1.35) (end 0.625 -2.35) (layer "F.Fab") (width 0.1))
     (pad "" np_thru_hole circle (at -1.6 2) (size 1.2 1.2) (drill 1.2) (layers *.Cu *.Mask))
-    (pad "1" thru_hole roundrect (at 0 0) (size 1.7 1.95) (drill 0.95) (layers *.Cu *.Mask) (roundrect_rratio 0.147059)
+    (pad "1" thru_hole roundrect (at 0 0) (size 1.7 1.95) (drill 0.95) (layers *.Cu *.Mask) (roundrect_rratio 0.1470588235)
       (net 20 "GND") (pinfunction "Pin_1") (pintype "passive"))
     (pad "2" thru_hole oval (at 2.5 0) (size 1.7 1.95) (drill 0.95) (layers *.Cu *.Mask)
@@
     (fp_line (start 12.45 3.4) (end 12.45 -2.35) (layer "F.Fab") (width 0.1))
     (pad "" np_thru_hole circle (at -1.6 2) (size 1.2 1.2) (drill 1.2) (layers *.Cu *.Mask))
-    (pad "1" thru_hole roundrect (at 0 0) (size 1.7 1.95) (drill 0.95) (layers *.Cu *.Mask) (roundrect_rratio 0.147059)
+    (pad "1" thru_hole roundrect (at 0 0) (size 1.7 1.95) (drill 0.95) (layers *.Cu *.Mask) (roundrect_rratio 0.1470588235)
       (net 2 "+5V") (pinfunction "Pin_1") (pintype "passive"))
     (pad "2" thru_hole oval (at 2.5 0) (size 1.7 1.95) (drill 0.95) (layers *.Cu *.Mask)
@@
     (fp_line (start 4.95 -2.35) (end -2.45 -2.35) (layer "F.Fab") (width 0.1))
     (pad "" np_thru_hole circle (at -1.6 2) (size 1.2 1.2) (drill 1.2) (layers *.Cu *.Mask))
-    (pad "1" thru_hole roundrect (at 0 0) (size 1.7 2) (drill 1) (layers *.Cu *.Mask) (roundrect_rratio 0.147059)
+    (pad "1" thru_hole roundrect (at 0 0) (size 1.7 2) (drill 1) (layers *.Cu *.Mask) (roundrect_rratio 0.1470588235)
       (net 20 "GND") (pinfunction "Pin_1") (pintype "passive"))
     (pad "2" thru_hole oval (at 2.5 0) (size 1.7 2) (drill 1) (layers *.Cu *.Mask)
@@
     (fp_line (start 14.95 3.4) (end 14.95 -2.35) (layer "F.Fab") (width 0.1))
     (pad "" np_thru_hole circle (at -1.6 2) (size 1.2 1.2) (drill 1.2) (layers *.Cu *.Mask))
-    (pad "1" thru_hole roundrect (at 0 0) (size 1.7 1.95) (drill 0.95) (layers *.Cu *.Mask) (roundrect_rratio 0.147059)
+    (pad "1" thru_hole roundrect (at 0 0) (size 1.7 1.95) (drill 0.95) (layers *.Cu *.Mask) (roundrect_rratio 0.1470588235)
       (net 78 "TOF2_EXTI") (pinfunction "Pin_1") (pintype "passive"))
     (pad "2" thru_hole oval (at 2.5 0) (size 1.7 1.95) (drill 0.95) (layers *.Cu *.Mask)
@@
     (fp_line (start -2.45 3.4) (end 7.45 3.4) (layer "F.Fab") (width 0.1))
     (pad "" np_thru_hole circle (at -1.6 2) (size 1.2 1.2) (drill 1.2) (layers *.Cu *.Mask))
-    (pad "1" thru_hole roundrect (at 0 0) (size 1.7 1.95) (drill 0.95) (layers *.Cu *.Mask) (roundrect_rratio 0.147059)
+    (pad "1" thru_hole roundrect (at 0 0) (size 1.7 1.95) (drill 0.95) (layers *.Cu *.Mask) (roundrect_rratio 0.1470588235)
       (net 20 "GND") (pinfunction "Pin_1") (pintype "passive"))
     (pad "2" thru_hole oval (at 2.5 0) (size 1.7 1.95) (drill 0.95) (layers *.Cu *.Mask)
@@
     (fp_line (start -2.45 -2.35) (end -2.45 3.4) (layer "F.Fab") (width 0.1))
     (pad "" np_thru_hole circle (at -1.6 2 270) (size 1.2 1.2) (drill 1.2) (layers *.Cu *.Mask))
-    (pad "1" thru_hole roundrect (at 0 0 270) (size 1.7 1.95) (drill 0.95) (layers *.Cu *.Mask) (roundrect_rratio 0.147059)
+    (pad "1" thru_hole roundrect (at 0 0 270) (size 1.7 1.95) (drill 0.95) (layers *.Cu *.Mask) (roundrect_rratio 0.1470588235)
       (net 4 "O1_D2") (pinfunction "Pin_1") (pintype "passive"))
     (pad "2" thru_hole oval (at 2.5 0 270) (size 1.7 1.95) (drill 0.95) (layers *.Cu *.Mask)
@@
   (gr_line (start 8 118) (end 8 116) (layer "F.Fab") (width 0.1))
   (gr_line (start 8 117) (end 8 118) (layer "F.Fab") (width 0.1))
+  (gr_text "Beerator\nA.P" (at 139.2 91.6) (layer "In1.Cu")
+    (effects (font (size 1.5 1.5) (thickness 0.3)))
+  )
   (segment (start 124.8 86.8) (end 126.6 85) (width 1) (layer "F.Cu") (net 1))
   (segment (start 114 81.4625) (end 112.45 81.4625) (width 1) (layer "F.Cu") (net 1))

Commit message: Correction Carte
Routing:
- net +5V: track 15.9 -> 19.0 mm
Changed lines of the file:
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@@
   (segment (start 136.26 68.09) (end 136.095 67.925) (width 0.3) (layer "F.Cu") (net 2))
   (segment (start 114.3 83.3625) (end 116.2 81.4625) (width 0.3) (layer "F.Cu") (net 2))
+  (segment (start 122.95 80.553249) (end 122.95 80.9375) (width 0.25) (layer "F.Cu") (net 2))
   (segment (start 136.26 70.85) (end 136.26 68.09) (width 0.3) (layer "F.Cu") (net 2))
+  (segment (start 121.05 80.9375) (end 121.05 80.553249) (width 0.25) (layer "F.Cu") (net 2))
+  (segment (start 122.346751 79.95) (end 122.95 80.553249) (width 0.25) (layer "F.Cu") (net 2))
+  (segment (start 121.05 80.553249) (end 121.653249 79.95) (width 0.25) (layer "F.Cu") (net 2))
+  (segment (start 121.653249 79.95) (end 122.346751 79.95) (width 0.25) (layer "F.Cu") (net 2))
   (segment (start 114.3 84.65) (end 114.3 83.3625) (width 0.3) (layer "F.Cu") (net 2))
   (via (at 151 59.8) (size 0.8) (drill 0.4) (layers "F.Cu" "B.Cu") (free) (net 2))
