File: KiCad/Beerator/Beerator.kicad_pcb (KiCad board)
At the start: 4 copper layers, 112 x 52 mm, 56 parts, among them SW201 SW_DPDT_x2, U201 REG-5, Y301 Crystal_GND23

Commit message: Kicad Changes
Routing:
- net +5V: track 19.0 -> 15.9 mm
- net +BATT: track 277.4 -> 276.5 mm
Changed lines of the file:
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@@
   (segment (start 122.6 93.8) (end 60.4 93.8) (width 1) (layer "F.Cu") (net 1))
   (segment (start 58.8 60.4) (end 59.2 60.4) (width 1) (layer "F.Cu") (net 1))
-  (segment (start 119.05 84.6) (end 118.5 84.05) (width 0.3) (layer "F.Cu") (net 1))
   (segment (start 59.6 60.4) (end 58.8 60.4) (width 0.75) (layer "F.Cu") (net 1))
   (segment (start 126.6 85) (end 149.4 85) (width 1) (layer "F.Cu") (net 1))
@@
   (segment (start 124.8 86.8) (end 122.65 84.65) (width 1) (layer "F.Cu") (net 1))
   (segment (start 92.4 56.2) (end 96.8625 56.2) (width 0.75) (layer "F.Cu") (net 1))
-  (segment (start 113.9 81.5625) (end 114 81.4625) (width 1) (layer "F.Cu") (net 1))
   (segment (start 72.244888 56.2) (end 92.4 56.2) (width 0.75) (layer "F.Cu") (net 1))
   (segment (start 63.644888 64.8) (end 63.644888 64.444888) (width 0.75) (layer "F.Cu") (net 1))
@@
   (segment (start 136.26 68.09) (end 136.095 67.925) (width 0.3) (layer "F.Cu") (net 2))
   (segment (start 114.3 83.3625) (end 116.2 81.4625) (width 0.3) (layer "F.Cu") (net 2))
-  (segment (start 122.95 80.553249) (end 122.95 80.9375) (width 0.25) (layer "F.Cu") (net 2))
   (segment (start 136.26 70.85) (end 136.26 68.09) (width 0.3) (layer "F.Cu") (net 2))
-  (segment (start 121.05 80.9375) (end 121.05 80.553249) (width 0.25) (layer "F.Cu") (net 2))
-  (segment (start 122.346751 79.95) (end 122.95 80.553249) (width 0.25) (layer "F.Cu") (net 2))
-  (segment (start 121.05 80.553249) (end 121.653249 79.95) (width 0.25) (layer "F.Cu") (net 2))
-  (segment (start 121.653249 79.95) (end 122.346751 79.95) (width 0.25) (layer "F.Cu") (net 2))
   (segment (start 114.3 84.65) (end 114.3 83.3625) (width 0.3) (layer "F.Cu") (net 2))
   (via (at 151 59.8) (size 0.8) (drill 0.4) (layers "F.Cu" "B.Cu") (free) (net 2))
@@
     (polygon
       (pts
-        (xy 163.2 105.8)
-        (xy 38 106.2)
-        (xy 38 37.8)
-        (xy 162 37.6)
+        (xy 163.199814 105.284516)
+        (xy 37.999814 105.684516)
+        (xy 37.999814 37.284516)
+        (xy 161.999814 37.084516)
       )
     )
